Commit message: ``` feat(urdf): 更新AM-D02机器人URDF模型参数
更新了多个关节的旋转轴方向、连杆惯性参数和几何变换矩阵，
包括左臂和右臂的关节配置，并修正了末端执行器的坐标系。

fix(config): 调整机器人关节力矩限制和安全限位参数

将第5、6关节的力矩限制从9.0调整为7.0，添加了完整的单臂参考
关节安全限位配置，并修改了初始姿态配置。

refactor(sim_env): 实现配置化的关节限位约束处理

重构关节限位逻辑，从使用MuJoCo模型原始限位改为使用配置文件
中的统一限位参数，并在初始化时应用到模型中。

perf(stm32): 优化控制周期并更新硬件配置参数

将控制步长从0.01s优化至0.001s，同步更新了关节力矩限制和
位置限位参数，修正了重力向量方向。

feat(model_lib): 重构AM-D02机器人动力学模型参数

重新定义了AM-D02机器人的DH参数、连杆质量和惯性矩阵等动力学
参数，更新了模型构建函数以支持新的物理参数。
```

File: AM-DPBSURDF0422/urdf/AM-DPBSURDF0422.urdf (robot description, URDF)
Before this commit: robot AM-DPBSURDF0422, 20 links, 18 joints
Joints:
- joint AM-D02-J14_Joint: axis 0 0 1 -> 0 0 -1
- joint AM-D02R-J03_Joint: axis 0 0 1 -> 0 0 -1
- joint ArmL04_Joint: axis 0 0 -1 -> 0 0 1
- joint ArmL06_Joint: axis 0 0 1 -> 0 0 -1
- joint ArmR01_Joint: axis 0 0 1 -> 0 0 -1
- joint ArmR04_Joint: axis 0 0 -1 -> 0 0 1
- joint ArmR05_Link: axis 0 0 -1 -> 0 0 1
- joint ArmR07Output_Link: axis 0 0 -1 -> 0 0 1

Commit message: ``` feat(urdf): 更新双臂URDF模型支持14轴控制
更新AM-DPBSURDF0422 URDF文件以支持左右双臂14轴联合控制，
调整了多个关节的轴向定义(xyz="0 0 -1"改为"0 0 1"或相反)，
修复了关节命名错误，并添加了右侧手臂的相关关节配置。

docs(readme): 更新文档说明双臂14轴仿真功能

将README文档中的描述从单臂7轴更新为双臂14轴仿真系统，
详细说明了新的UDP通信协议格式，包括43个double输入和14个
double输出的数据结构，并添加了AM_D02_FIX_UNCONTROLLED_JOINTS
环境变量说明。

refactor(c_interface): 重构C接口支持双臂14轴控制

修改C接口代码以支持14轴双臂控制，更新了状态变量数组大小，
调整了扭矩输出处理逻辑，修改了UDP通信数据包格式以包含
左右臂目标位置和姿态信息。

feat(sim_bridge): 添加双臂独立控制桥接功能

扩展sim_bridge模块以支持左右臂独立控制，新增
control_step_v2_mujoco_arm函数来处理指定侧臂的控制逻辑，
更新了函数签名以适应14轴输入输出。

refactor(sim_interface): 重构仿真接口适配双臂协议

更新仿真接口的UDP通信协议，将数据包格式从2个double
扩展到43个double，支持双臂关节状态和目标姿态传输，
相应更新了数据解析和发送逻辑。

feat(config): 配置系统升级支持双臂14轴仿真

更新Python配置模块以支持双臂14轴仿真，添加了左右臂
关节名称列表、扭矩限制、安全限位等独立配置参数，
并提供了TCP偏移量和坐标系转换的双臂支持。
```

File: AM-DPBSURDF0422/urdf/AM-DPBSURDF0422.urdf (robot description, URDF)
Before this commit: robot AM-DPBSURDF0422, 20 links, 18 joints
Joints:
- joint AM-D02-J14_Joint: axis 0 0 -1 -> 0 0 1
- joint AM-D02R-J03_Joint: axis 0 0 -1 -> 0 0 1; limit lower=-0.26 upper=2.26 effort=40 velocity=0 -> lower=-0.6605 upper=2.203 effort=40 velocity=0
- joint ArmL04_Joint: axis 0 0 1 -> 0 0 -1
- joint ArmL06_Joint: axis 0 0 -1 -> 0 0 1
- joint ArmL07Output_Joint: origin xyz=0 -0.0204999999999969 -0.0374999999999962 rpy=1.57079632678463 1.5707963267949 0 -> xyz=0 -0.0204999999999969 -0.0374999999999962 rpy=1.57079632678463 4.71238898038469 0
- joint ArmL07_Joint: axis 0 0 -1 -> 0 0 1
- joint ArmR01_Joint: axis 0 0 -1 -> 0 0 1; limit lower=-2.35 upper=2.35 effort=40 velocity=0 -> lower=-2.405 upper=2.2175 effort=40 velocity=0
- joint ArmR04_Joint: axis 0 0 1 -> 0 0 -1; limit lower=-1.65 upper=1.65 effort=27 velocity=0 -> lower=-1.763 upper=1.594 effort=27 velocity=0
- joint ArmR05_Link: limit lower=-2.268 upper=0 effort=27 velocity=0 -> lower=-0.0165 upper=2.3235 effort=27 velocity=0
- joint ArmR06_Link: axis 0 0 -1 -> 0 0 1; limit lower=-1.57 upper=1.57 effort=9 velocity=0 -> lower=-1.5935 upper=1.574 effort=9 velocity=0
- joint ArmR07Output_Link: axis 0 0 1 -> 0 0 -1; limit lower=-1.37 upper=1.57 effort=9 velocity=0 -> lower=-1.1075 upper=1.068 effort=9 velocity=0
- joint ArmR07_Link: axis 0 0 -1 -> 0 0 1; limit lower=-0.724 upper=1.06 effort=9 velocity=0 -> lower=-0.6015 upper=0.6755 effort=9 velocity=0
